Commit message: camera_interface.py

File: drone_basic/urdf/hector_camera_laser.urdf.xacro (robot description, xacro)
@@ -13,10 +13,5 @@
                           cam_info_topic="front_cam/camera_info" update_rate="10" res_x="1280" res_y="1080"
                           image_format="R8G8B8" hfov="90">
-      <origin xyz="0.4 0 0 " rpy="0 0 0"/>
-    </xacro:generic_camera>
-    <xacro:generic_camera name="down_cam" parent="base_link" ros_topic="down_cam/image"
-                          cam_info_topic="down_cam/camera_info" update_rate="10" res_x="1280" res_y="1080"
-                          image_format="R8G8B8" hfov="90">
-      <origin xyz="0 0 -0.14" rpy="0 1.57 0"/>
+      <origin xyz="0.4 0 0 " rpy="0 0.57 0"/>
     </xacro:generic_camera>
     <xacro:include filename="$(find hector_quadrotor_gazebo)/urdf/quadrotor_plugins.gazebo.xacro" />

File: drone_basic/urdf/quadrotor_base.urdf.xacro (robot description, xacro)
@@ -25,5 +25,5 @@
     </link>
     <!-- Sonar height sensor -->
-    <xacro:sonar_sensor name="sonar" parent="base_link" ros_topic="sonar_height" update_rate="10" min_range="0.03" max_range="3.0" field_of_view="${40*pi/180}" ray_count="3">
+    <xacro:sonar_sensor name="sonar" parent="base_link" ros_topic="sonar_height" update_rate="10" min_range="0.03" max_range="6.0" field_of_view="${40*pi/180}" ray_count="3">
       <origin xyz="-0.16 0.0 -0.012" rpy="0 ${90*pi/180} 0"/>
     </xacro:sonar_sensor>
